File: Kicad/2m pieper THT.kicad_pcb (KiCad board)
At the start: 2 copper layers, 90 x 90 mm, 80 parts, among them J1 AUX, J3 RF, J4 RF, J5 JQ8400-FL, J6 BATTERY, J7 SWITCH, Q1 BFR193, Q2 BFR193, Q3 ZVP2106A, SW1 SW_Push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

Commit message: Added files
Parts:
- J2: value ~ -> 1x3 header
Changed lines of the file:
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@@
 	)
 	(paper "A4")
+	(title_block
+		(title "iPieper")
+		(date "2025-04-22")
+		(rev "1")
+		(company "PE5PVB")
+	)
 	(layers
 		(0 "F.Cu" signal)
@@
 			)
 		)
-		(property "Value" "~"
+		(property "Value" "1x3 header"
 			(at 0 7.41 0)
 			(layer "F.Fab")

Commit message: Update data
Parts:
- R13: value 82 -> 47
- R14: value 47 -> 82
- R9: value 47 -> 10
Other:
- board text added: "G"
- board text added: "k"
- board text removed: "L"
Changed lines of the file:
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@@
 			)
 		)
-		(property "Value" "47"
+		(property "Value" "82"
 			(at 5.08 2.37 0)
 			(layer "F.Fab")
@@
 			)
 		)
-		(property "Value" "82"
+		(property "Value" "47"
 			(at 5.08 2.37 90)
 			(layer "F.Fab")
@@
 			)
 		)
-		(property "Value" "47"
+		(property "Value" "10"
 			(at 5.08 2.37 0)
 			(layer "F.Fab")
@@
 		)
 	)
+	(gr_text "G"
+		(at 182.8292 91.0082 0)
+		(layer "F.SilkS")
+		(effects
+			(font
+				(size 1 1)
+				(thickness 0.15)
+			)
+			(justify left bottom)
+		)
+	)
 	(gr_text "Radiokampweek 2025"
 		(at 201.9808 115.57 0)
@@
 		)
 	)
-	(gr_text "L"
+	(gr_text "k"
 		(at 165.735 102.6668 0)
 		(layer "F.SilkS")

Commit message: Modificaties
Parts:
- C15, C19: value 47n -> 10n
- C16: value 47n -> 27p
- C17: value 100p -> 27p
- C21: value 22p -> 27p
- C3: value 6n8 -> 1uF
- C8: value 1n -> 27p
- R1: value 2k -> 10k
- R14: value 82 -> 47
- R9: value 10 -> 22
Changed lines of the file:
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@@
 			)
 		)
-		(property "Value" "82"
+		(property "Value" "47"
 			(at 5.08 2.37 0)
 			(layer "F.Fab")
@@
 			)
 		)
-		(property "Value" "100p"
+		(property "Value" "27p"
 			(at 1.25 2.25 90)
 			(layer "F.Fab")
@@
 			)
 		)
-		(property "Value" "2k"
+		(property "Value" "10k"
 			(at 5.08 2.37 0)
 			(layer "F.Fab")
@@
 			)
 		)
-		(property "Value" "1n"
+		(property "Value" "27p"
 			(at 1.25 2.25 90)
 			(layer "F.Fab")
@@
 			)
 		)
-		(property "Value" "10"
+		(property "Value" "22"
 			(at 5.08 2.37 0)
 			(layer "F.Fab")
@@
 			)
 		)
-		(property "Value" "22p"
+		(property "Value" "27p"
 			(at 1.25 2.25 0)
 			(layer "F.Fab")
@@
 			)
 		)
-		(property "Value" "47n"
+		(property "Value" "27p"
 			(at 1.25 2.25 90)
 			(layer "F.Fab")
@@
 			)
 		)
-		(property "Value" "47n"
+		(property "Value" "10n"
 			(at 1.25 2.25 90)
 			(layer "F.Fab")
@@
 			)
 		)
-		(property "Value" "47n"
+		(property "Value" "10n"
 			(at 1.25 2.25 0)
 			(layer "F.Fab")
@@
 			)
 		)
-		(property "Value" "6n8"
+		(property "Value" "1uF"
 			(at 1.25 2.25 90)
 			(layer "F.Fab")
