File: Kicad/2m pieper THT.kicad_sch (KiCad schematic)
At the start: 79 parts, among them J1 AUX, J3 RF, J4 RF, J5 JQ8400-FL, J6 BATTERY, J7 SWITCH, Q1 BFR193, Q2 BFR193, Q3 ZVP2106A, SW1 SW_Push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

Commit message: Added files
Parts:
- J2: value ~ -> 1x3 header
Other:
- company: (none) -> PE5PVB
- title: (none) -> iPieper
Changed lines of the file:
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@@
 	(generator_version "9.0")
 	(paper "A4")
+	(title_block
+		(title "iPieper")
+		(date "2025-04-22")
+		(rev "1")
+		(company "PE5PVB")
+	)
 	(text "L5 + L7: 3 windingen, 9mm diameter, 9mm lengte\nL6: 4 windingen, 9mm diameter, 9mm lengte"
 		(exclude_from_sim no)
@@
 			)
 		)
-		(property "Value" "~"
+		(property "Value" "1x3 header"
 			(at 99.06 104.14 90)
 			(effects
@@
 				)
 				(justify right)
+				(hide yes)
 			)
 		)

Commit message: Update data
Parts:
- R13: value 82 -> 47
- R14: value 47 -> 82
- R9: value 47 -> 10
Changed lines of the file:
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@@
 			)
 		)
-		(property "Value" "47"
+		(property "Value" "82"
 			(at 128.905 65.405 0)
 			(effects
@@
 			)
 		)
-		(property "Value" "82"
+		(property "Value" "47"
 			(at 128.905 38.735 0)
 			(effects
@@
 		(on_board yes)
 		(dnp no)
-		(fields_autoplaced yes)
 		(property "Reference" "R9"
-			(at 96.52 62.865 0)
+			(at 95.885 62.865 0)
 			(effects
 				(font
@@
 			)
 		)
-		(property "Value" "47"
-			(at 96.52 65.405 0)
+		(property "Value" "10"
+			(at 95.885 65.405 0)
 			(effects
 				(font

Commit message: Update
Other:
- note added: "L5 + L7: 3 windingen, 7mm diameter, 9mm lengte L6: 4 windingen, 7mm diameter, 9mm lengte"
- note removed: "L5 + L7: 3 windingen, 9mm diameter, 9mm lengte L6: 4 windingen, 9mm diameter, 9mm lengte"
Changed lines of the file:
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@@
 		(company "PE5PVB")
 	)
-	(text "L5 + L7: 3 windingen, 9mm diameter, 9mm lengte\nL6: 4 windingen, 9mm diameter, 9mm lengte"
+	(text "L5 + L7: 3 windingen, 7mm diameter, 9mm lengte\nL6: 4 windingen, 7mm diameter, 9mm lengte"
 		(exclude_from_sim no)
 		(at 140.97 39.37 0)

Commit message: Modificaties
Parts:
- C15, C19: value 47n -> 10n
- C16: value 47n -> 27p
- C17: value 100p -> 27p
- C21: value 22p -> 27p
- C3: value 6n8 -> 1uF
- C8: value 1n -> 27p
- R1: value 2k -> 10k
- R14: value 82 -> 47
- R9: value 10 -> 22
Changed lines of the file:
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@@
 			)
 		)
-		(property "Value" "82"
+		(property "Value" "47"
 			(at 128.905 65.405 0)
 			(effects
@@
 		(on_board yes)
 		(dnp no)
-		(fields_autoplaced yes)
 		(property "Reference" "C19"
-			(at 136.525 62.8713 0)
+			(at 137.16 62.865 0)
 			(effects
 				(font
@@
 			)
 		)
-		(property "Value" "47n"
-			(at 136.525 65.4113 0)
+		(property "Value" "10n"
+			(at 137.16 65.405 0)
 			(effects
 				(font
@@
 			)
 		)
-		(property "Value" "22p"
+		(property "Value" "27p"
 			(at 138.4363 45.72 90)
 			(effects
@@
 			)
 		)
-		(property "Value" "100p"
+		(property "Value" "27p"
 			(at 106.68 57.15 0)
 			(effects
@@
 			)
 		)
-		(property "Value" "6n8"
+		(property "Value" "1uF"
 			(at 15.875 112.395 0)
 			(effects
@@
 			)
 		)
-		(property "Value" "2k"
+		(property "Value" "10k"
 			(at 15.875 92.71 0)
 			(effects
@@
 		(on_board yes)
 		(dnp no)
-		(fields_autoplaced yes)
 		(property "Reference" "C16"
-			(at 105.4163 43.18 90)
+			(at 105.41 43.18 90)
 			(effects
 				(font
@@
 			)
 		)
-		(property "Value" "47n"
-			(at 105.4163 45.72 90)
+		(property "Value" "27p"
+			(at 105.41 45.72 90)
 			(effects
 				(font
@@
 			)
 		)
-		(property "Value" "1n"
+		(property "Value" "27p"
 			(at 54.6163 45.085 90)
 			(effects
@@
 		(on_board yes)
 		(dnp no)
-		(fields_autoplaced yes)
 		(property "Reference" "C15"
-			(at 103.505 62.8713 0)
+			(at 104.14 62.865 0)
 			(effects
 				(font
@@
 			)
 		)
-		(property "Value" "47n"
-			(at 103.505 65.4113 0)
+		(property "Value" "10n"
+			(at 104.14 65.405 0)
 			(effects
 				(font
@@
 			)
 		)
-		(property "Value" "10"
+		(property "Value" "22"
 			(at 95.885 65.405 0)
 			(effects
